Commit message: 修改雷达参数和frame

File: nav2_bringup/tarkbot_model/tarkbot_car_laser.urdf.xacro (robot description, xacro)
@@ -45,5 +45,5 @@
     <xacro:property name="laser_m" value="0.1" /> <!-- 雷达质量 -->
     <!-- 雷达关节以及link -->
-    <link name="laser_link">
+    <link name="base_scan">
         <visual>
             <geometry>
@@ -67,8 +67,8 @@
     <joint name="laser_base_link" type="fixed">
         <parent link="support" />
-        <child link="laser_link" />
+        <child link="base_scan" />
         <origin xyz="${laser_x} ${laser_y} ${laser_z}" />
     </joint>
-    <gazebo reference="laser_link">
+    <gazebo reference="base_scan">
         <material>Gazebo/Black</material>
     </gazebo>

File: nav2_bringup/tarkbot_model/tarkbot_lidar_sensor.urdf.xacro (robot description, xacro)
@@ -1,9 +1,9 @@
 <robot name="my_sensors" xmlns:xacro="http://wiki.ros.org/xacro">
   <!-- 雷达 -->
-  <gazebo reference="laser_link">
-    <sensor type="gpu_ray" name="rplidar">
+  <gazebo reference="base_scan">
+    <sensor type="ray" name="rplidar">
       <pose>0 0 0 0 0 0</pose>
       <visualize>true</visualize>
-      <update_rate>10</update_rate>
+      <update_rate>5</update_rate>
       <ray>
         <scan>
@@ -11,12 +11,12 @@
             <samples>360</samples>
             <resolution>1</resolution>
-            <min_angle>-3.1415926</min_angle>
-            <max_angle>3.1415926</max_angle>
+            <min_angle>0.000000</min_angle>
+            <max_angle>6.280000</max_angle>
           </horizontal>
         </scan>
         <range>
-          <min>0.20</min>
-          <max>30.0</max>
-          <resolution>0.01</resolution>
+          <min>0.120000</min>
+          <max>20.0</max>
+          <resolution>0.015000</resolution>
         </range>
         <noise>
@@ -26,11 +26,10 @@
         </noise>
       </ray>
-      <plugin name="gazebo_rplidar" filename="libgazebo_ros_ray_sensor.so">
+      <plugin name="tarkbot_laserscan" filename="libgazebo_ros_ray_sensor.so">
         <ros>
-          <namespace>/</namespace>
           <remapping>~/out:=scan</remapping>
         </ros>
         <output_type>sensor_msgs/LaserScan</output_type>
-        <frame_name>laser_link</frame_name>
+        <frame_name>base_scan</frame_name>
       </plugin>
     </sensor>
