Commit message: 添加tarkbot小车的阿克曼仿真模型，可以通过/ackermann_steering_controller/reference控制

File: nav2_bringup/tarkbot_model/tarkbot_car_base.urdf.xacro (robot description, xacro)
@@ -8,93 +8,153 @@
 <!-- 根标签，必须声明 xmlns:xacro -->
 <robot name="my_base" xmlns:xacro="http://www.ros.org/wiki/xacro">
-    <!-- 封装变量、常量 -->
-    <!-- PI 值设置精度需要高一些，否则后续车轮翻转量计算时，可能会出现肉眼不能察觉的车轮倾斜，从而导致模型抖动 -->
-    <xacro:property name="PI" value="3.1415926"/>
-    <!-- 宏:黑色设置 -->
-    <material name="black">
-        <color rgba="0.0 0.0 0.0 1.0" />
-    </material>
-    <!-- 底盘属性 -->
-    <xacro:property name="base_footprint_radius" value="0.001" /> <!-- base_footprint 半径  -->
-    <!--<xacro:property name="base_link_radius" value="0.1" />  base_link 半径 -->
-    <!--<xacro:property name="base_link_length" value="0.08" />  base_link 长 -->
-    <xacro:property name="base_link_length" value="0.2" />  <!--base_link 长  -->
-    <xacro:property name="base_link_width" value="0.1" />  <!--base_link 宽 -->
-    <xacro:property name="base_link_height" value="0.05" />  <!--base_link 高 -->
-    <xacro:property name="earth_space" value="0.055" /> <!-- 离地间距 -->
-    <xacro:property name="base_link_m" value="2.0" /> <!-- 质量  -->
-    <!-- 底盘 -->
-    <link name="base_footprint">
+  <!-- 封装变量、常量 -->
+  <!-- PI 值设置精度需要高一些，否则后续车轮翻转量计算时，可能会出现肉眼不能察觉的车轮倾斜，从而导致模型抖动 -->
+  <xacro:property name="PI" value="3.1415926" />
+  <!-- 宏:黑色设置 -->
+  <material name="black">
+    <color rgba="0.0 0.0 0.0 1.0" />
+  </material>
+  <material name="green">
+    <color rgba="0.0 1.0 0.0 1.0" />
+  </material>
+  <!-- 底盘属性 -->
+  <xacro:property name="base_footprint_radius" value="0.001" /> <!-- base_footprint 半径  -->
+  <xacro:property name="base_link_length" value="0.2" />  <!--base_link
+  长  -->
+  <xacro:property name="base_link_width" value="0.1" />  <!--base_link
+  宽 -->
+  <xacro:property name="base_link_height" value="0.05" />  <!--base_link
+  高 -->
+  <xacro:property name="earth_space" value="0.055" /> <!-- 离地间距 -->
+  <xacro:property name="base_link_m" value="2.0" /> <!-- 质量  -->
+  <!-- 底盘 -->
+  <link name="base_footprint">
+    <visual>
+      <geometry>
+        <sphere radius="${base_footprint_radius}" />
+      </geometry>
+    </visual>
+  </link>
+  <link name="base_link">
+    <visual>
+      <geometry>
+        <box size="${base_link_length} ${base_link_width} ${base_link_height}" />
+      </geometry>
+      <origin xyz="0 0 0" rpy="0 0 0" />
+      <material name="black">
+        <color rgba="0.5 0.3 0.0 0.5" />
+      </material>
+    </visual>
+    <!-- <collision>
+      <geometry>
+        <box size="${base_link_length} ${base_link_width}-0.05 ${base_link_height}" />
+      </geometry>
+      <origin xyz="0 0 0" rpy="0 0 0" />
+    </collision> -->
+    <xacro:box_inertial_matrix m="${base_link_m}" l="${base_link_length}" w="${base_link_width}"
+      h="${base_link_height}" />
+  </link>
+  <gazebo reference="base_link">
+    <material>Gazebo/Green</material>
+  </gazebo>
+  <joint name="base_link2base_footprint" type="fixed">
+    <parent link="base_footprint" />
+    <child link="base_link" />
+    <origin xyz="0 0 ${earth_space + base_link_height / 2 }" />
+  </joint>
+  <!-- 驱动轮 -->
+  <!-- 驱动轮属性 -->
+  <xacro:property name="wheel_radius" value="0.03" /><!-- 半径 -->
+  <xacro:property name="wheel_length" value="0.02" /><!-- 宽度 -->
+  <xacro:property name="wheel_m" value="1.0" /> <!-- 质量  -->
+  <!-- 驱动轮宏实现 -->
+  <xacro:macro name="add_back_wheels" params="name1 name2 flag1 flag2">
+    <link name="${name1}_${name2}_wheel">
       <visual>
         <geometry>
-          <sphere radius="${base_footprint_radius}" />
+          <cylinder radius="${wheel_radius}" length="${wheel_length}" />
         </geometry>
-      </visual>
-    </link>
-    <link name="base_link">
-      <visual>
-        <geometry>
-          <box size="${base_link_length} ${base_link_width} ${base_link_height}" />
-          <!-- <cylinder radius="${base_link_radius}" length="${base_link_length}" /> -->
-        </geometry>
-        <origin xyz="0 0 0" rpy="0 0 0" />
-        <material name="black">
-          <color rgba="0.5 0.3 0.0 0.5" />
-        </material>
+        <origin xyz="0.0 0.0 0.0" rpy="${PI / 2} 0.0 0.0" />
+        <material name="black" />
       </visual>
       <collision>
         <geometry>
-          <box size="${base_link_length} ${base_link_width} ${base_link_height}" />
-          <!-- <cylinder radius="${base_link_radius}" length="${base_link_length}" /> -->
+          <cylinder radius="${wheel_radius}" length="${wheel_length}" />
         </geometry>
-        <origin xyz="0 0 0" rpy="0 0 0" />
+        <origin xyz="0.0 0.0 0.0" rpy="${PI / 2} 0.0 0.0" />
       </collision>
-      <xacro:box_inertial_matrix m="${base_link_m}" l="${base_link_length}" w="${base_link_width}" h="${base_link_height}" />
-      <!-- <xacro:cylinder_inertial_matrix m="${base_link_m}" r="${base_link_radius}" h="${base_link_length}" /> -->
+      <xacro:cylinder_inertial_matrix m="${wheel_m}" r="${wheel_radius}" h="${wheel_length}" />
     </link>
-    <joint name="base_link2base_footprint" type="fixed">
-      <parent link="base_footprint" />
-      <child link="base_link" />
-      <origin xyz="0 0 ${earth_space + base_link_height / 2 }" />
+    <joint name="${name1}_${name2}_wheel_joint" type="continuous">
+      <parent link="base_link" />
+      <child link="${name1}_${name2}_wheel" />
+      <origin
+        xyz="
+        ${flag2 * (base_link_length/2 - 0.015 - wheel_radius)}
+        ${flag1 * (base_link_width/2 + wheel_length/2)}
+        ${(wheel_radius - earth_space ) }"
+      />
+      <axis xyz="0 1 0" />
     </joint>
-    <gazebo reference="base_link">
-        <material>Gazebo/Blue</material>
+    <gazebo reference="${name1}_${name2}_wheel">
+      <material>Gazebo/Red</material>
     </gazebo>
-    <!-- 驱动轮 -->
-    <!-- 驱动轮属性 -->
-    <xacro:property name="wheel_radius" value="0.03" /><!-- 半径 -->
-    <xacro:property name="wheel_length" value="0.02" /><!-- 宽度 -->
-    <xacro:property name="wheel_m" value="1.0" /> <!-- 质量  -->
-    <!-- 驱动轮宏实现 -->
-    <xacro:macro name="add_wheels" params="name1 name2 flag1 flag2">
-      <link name="${name1}_${name2}_wheel">
-        <visual>
-          <geometry>
-            <cylinder radius="${wheel_radius}" length="${wheel_length}" />
-          </geometry>
-          <origin xyz="0.0 0.0 0.0" rpy="${PI / 2} 0.0 0.0" />
-          <material name="black" />
-        </visual>
-        <collision>
-          <geometry>
-            <cylinder radius="${wheel_radius}" length="${wheel_length}" />
-          </geometry>
-          <origin xyz="0.0 0.0 0.0" rpy="${PI / 2} 0.0 0.0" />
-        </collision>
-        <xacro:cylinder_inertial_matrix m="${wheel_m}" r="${wheel_radius}" h="${wheel_length}" />
-      </link>
-      <joint name="${name1}_${name2}_wheel_base_link" type="continuous">
-        <parent link="base_link" />
-        <child link="${name1}_${name2}_wheel" />
-        <origin xyz="${flag2 * (base_link_length/2 - 0.015 - wheel_radius)} ${flag1 * (base_link_width/2 + wheel_length/2)} ${(wheel_radius - earth_space ) }" />
-        <axis xyz="0 1 0" />
-      </joint>
-      <gazebo reference="${name1}_${name2}_wheel">
-        <material>Gazebo/Red</material>
-      </gazebo>
-    </xacro:macro>
-    <xacro:add_wheels name1="left" name2="front" flag1="1" flag2="1" />
-    <xacro:add_wheels name1="right" name2="front" flag1="-1" flag2="1" />
-    <xacro:add_wheels name1="left" name2="back" flag1="1" flag2="-1" />
-    <xacro:add_wheels name1="right" name2="back" flag1="-1" flag2="-1" />
+  </xacro:macro>
+  <!-- 前轮 -->
+  <xacro:macro name="add_front_wheels" params="name1 name2 flag1 flag2">
+    <!-- 转向机构 -->
+    <link name="${name1}_${name2}_wheel_steering">
+      <inertial>
+        <mass value="0.1" />
+        <inertia ixx="0.1" ixy="0.0" ixz="0.0" iyy="0.1" iyz="0.0" izz="0.1" />
+      </inertial>
+    </link>
+    <!-- 0.005为留点空间给前轮转向 -->
+    <joint name="${name1}_${name2}_steering_joint" type="revolute">
+      <parent link="base_link" />
+      <child link="${name1}_${name2}_wheel_steering" />
+      <axis xyz="0 1 0" />
+      <origin
+        xyz="
+        ${flag2 * (base_link_length/2 - 0.015 - wheel_radius)}
+        ${flag1 * (base_link_width/2 + wheel_length/2 + 0.005)}
+        ${(wheel_radius - earth_space ) }"
+        rpy="${PI / 2} 0.0 0.0"
+      />
+      <dynamics damping="0.2" />
+      <limit effort="1000" lower="${-PI}" upper="${PI}" velocity="30" />
+    </joint>
+    <!-- 轮子 -->
+    <link name="${name1}_${name2}_wheel">
+      <visual>
+        <geometry>
+          <cylinder radius="${wheel_radius}" length="${wheel_length}" />
+        </geometry>
+        <material name="green" />
+      </visual>
+      <collision>
+        <geometry>
+          <cylinder radius="${wheel_radius}" length="${wheel_length}" />
+        </geometry>
+      </collision>
+      <xacro:cylinder_inertial_matrix m="${wheel_m}" r="${wheel_radius}" h="${wheel_length}" />
+    </link>
+    <joint name="${name1}_${name2}_wheel_joint" type="continuous">
+      <parent link="${name1}_${name2}_wheel_steering" />
+      <child link="${name1}_${name2}_wheel" />
+      <origin xyz="0.0 0.0 0.0" rpy="0.0 0.0 0.0" />
+      <axis xyz="0 0 1" />
+      <dynamics damping="0.2" />
+    </joint>
+    <gazebo reference="${name1}_${name2}_wheel">
+      <material>Gazebo/Yellow</material>
+    </gazebo>
+    <gazebo reference="${name1}_${name2}_wheel_steering">
+      <material>Gazebo/Black</material>
+    </gazebo>
+  </xacro:macro>
+  <xacro:add_front_wheels name1="left" name2="front" flag1="1" flag2="1" />
+  <xacro:add_front_wheels name1="right" name2="front" flag1="-1" flag2="1" />
+  <xacro:add_back_wheels name1="left" name2="back" flag1="1" flag2="-1" />
+  <xacro:add_back_wheels name1="right" name2="back" flag1="-1" flag2="-1" />
 </robot>

File: nav2_bringup/tarkbot_model/tarkbot_move.urdf.xacro (robot description, xacro)
@@ -1,47 +1,32 @@
 <robot name="my_car_move" xmlns:xacro="http://wiki.ros.org/xacro">
-    <!-- 传动实现:用于连接控制器与关节 -->
-    <xacro:macro name="joint_trans" params="joint_name">
-        <!-- Transmission is important to link the joints and the controller -->
-        <transmission name="${joint_name}_trans">
-            <type>transmission_interface/SimpleTransmission</type>
-            <joint name="${joint_name}">
-                <hardwareInterface>hardware_interface/VelocityJointInterface</hardwareInterface>
-            </joint>
-            <actuator name="${joint_name}_motor">
-                <hardwareInterface>hardware_interface/VelocityJointInterface</hardwareInterface>
-                <mechanicalReduction>1</mechanicalReduction>
-            </actuator>
-        </transmission>
-    </xacro:macro>
-    <!-- 每一个驱动轮都需要配置传动装置 -->
-    <xacro:joint_trans joint_name="left_front_wheel_base_link" />
-    <xacro:joint_trans joint_name="right_front_wheel_base_link" />
-    <xacro:joint_trans joint_name="left_back_wheel_base_link" />
-    <xacro:joint_trans joint_name="right_back_wheel_base_link" />
-    <!-- 控制器 -->
-    <gazebo>
-        <plugin name="skid_steer_drive_controller" filename="libgazebo_ros_skid_steer_drive.so">
-            <rosDebugLevel>Debug</rosDebugLevel>
-            <publishWheelTF>true</publishWheelTF>
-            <robotNamespace></robotNamespace>
-            <publishTf>1</publishTf>
-            <publishWheelJointState>false</publishWheelJointState>
-            <alwaysOn>true</alwaysOn>
-            <updateRate>100.0</updateRate>\
-            <legacyMode>true</legacyMode>
-            <leftFrontJoint>left_front_wheel_base_link</leftFrontJoint> <!-- 左前轮 -->
-            <rightFrontJoint>right_front_wheel_base_link</rightFrontJoint> <!-- 右前轮 -->
-            <leftRearJoint>left_back_wheel_base_link</leftRearJoint> <!-- 左后轮 -->
-            <rightRearJoint>right_back_wheel_base_link</rightRearJoint> <!-- 右后轮 -->
-            <wheelSeparation>${base_link_width}</wheelSeparation> <!-- 车轮间距 -->
-            <wheelDiameter>${wheel_radius * 2}</wheelDiameter> <!-- 车轮直径 -->
-            <broadcastTF>1</broadcastTF>
-            <wheelTorque>30</wheelTorque>
-            <wheelAcceleration>1.8</wheelAcceleration>
-            <commandTopic>cmd_vel</commandTopic> <!-- 运动控制话题 -->
-            <odometryFrame>odom</odometryFrame>
-            <odometryTopic>odom</odometryTopic> <!-- 里程计话题 -->
-            <robotBaseFrame>/base_footprint</robotBaseFrame> <!-- 根坐标系 -->
-        </plugin>
-    </gazebo>
+  <ros2_control name="GazeboSimSystem" type="system">
+    <hardware>
+      <plugin>gazebo_ros2_control/GazeboSystem</plugin>
+    </hardware>
+    <joint name="left_back_wheel_joint">
+      <command_interface name="velocity" />
+      <state_interface name="velocity" />
+      <state_interface name="position" />
+    </joint>
+    <joint name="right_back_wheel_joint">
+      <command_interface name="velocity" />
+      <state_interface name="velocity" />
+      <state_interface name="position" />
+    </joint>
+    <joint name="left_front_steering_joint">
+      <command_interface name="position" />
+      <state_interface name="position" />
+    </joint>
+    <joint name="right_front_steering_joint">
+      <command_interface name="position" />
+      <state_interface name="position" />
+    </joint>
+  </ros2_control>
+  <gazebo>
+    <plugin name="gazebo_ros2_control" filename="libgazebo_ros2_control.so">
+      <parameters>
+        $(find nav2_bringup)/params/ackermann_drive_controller.yaml
+      </parameters>
+    </plugin>
+  </gazebo>
 </robot>

Commit message: 更换gazebo ackermann插件为gazebo_ros_pkg中的ackermann插件

File: nav2_bringup/tarkbot_model/tarkbot_car_base.urdf.xacro (robot description, xacro)
@@ -68,5 +68,5 @@
   <xacro:property name="wheel_length" value="0.02" /><!-- 宽度 -->
   <xacro:property name="wheel_m" value="1.0" /> <!-- 质量  -->
-  <!-- 驱动轮宏实现 -->
+  <!-- 后轮 -->
   <xacro:macro name="add_back_wheels" params="name1 name2 flag1 flag2">
     <link name="${name1}_${name2}_wheel">
@@ -75,5 +75,4 @@
           <cylinder radius="${wheel_radius}" length="${wheel_length}" />
         </geometry>
-        <origin xyz="0.0 0.0 0.0" rpy="${PI / 2} 0.0 0.0" />
         <material name="black" />
       </visual>
@@ -82,5 +81,4 @@
           <cylinder radius="${wheel_radius}" length="${wheel_length}" />
         </geometry>
-        <origin xyz="0.0 0.0 0.0" rpy="${PI / 2} 0.0 0.0" />
       </collision>
       <xacro:cylinder_inertial_matrix m="${wheel_m}" r="${wheel_radius}" h="${wheel_length}" />
@@ -94,6 +92,8 @@
         ${flag1 * (base_link_width/2 + wheel_length/2)}
         ${(wheel_radius - earth_space ) }"
+        rpy="${flag1 * PI/2} 0.0 0.0"
       />
-      <axis xyz="0 1 0" />
+      <axis xyz="0 0 ${-flag1}" />
+      <limit lower="-3.14159" upper="3.14159" effort="70" velocity="-1" />
     </joint>
     <gazebo reference="${name1}_${name2}_wheel">
@@ -114,5 +114,5 @@
       <parent link="base_link" />
       <child link="${name1}_${name2}_wheel_steering" />
-      <axis xyz="0 1 0" />
+      <axis xyz="0 0 1" />
       <origin
         xyz="
@@ -120,8 +120,7 @@
         ${flag1 * (base_link_width/2 + wheel_length/2 + 0.005)}
         ${(wheel_radius - earth_space ) }"
-        rpy="${PI / 2} 0.0 0.0"
+        rpy="0.0 0.0 0.0"
       />
-      <dynamics damping="0.2" />
-      <limit effort="1000" lower="${-PI}" upper="${PI}" velocity="30" />
+      <limit effort="-1" lower="${-PI}" upper="${PI}" velocity="-1" />
     </joint>
     <!-- 轮子 -->
@@ -144,6 +143,6 @@
       <child link="${name1}_${name2}_wheel" />
       <origin xyz="0.0 0.0 0.0" rpy="0.0 0.0 0.0" />
-      <axis xyz="0 0 1" />
-      <dynamics damping="0.2" />
+      <axis xyz="0 0 -1" />
+      <limit lower="-3.14159" upper="3.14159" effort="200" velocity="-1" />
     </joint>
     <gazebo reference="${name1}_${name2}_wheel">
@@ -158,3 +157,28 @@
   <xacro:add_back_wheels name1="left" name2="back" flag1="1" flag2="-1" />
   <xacro:add_back_wheels name1="right" name2="back" flag1="-1" flag2="-1" />
+  <!-- 虚拟方向盘 -->
+  <!-- Virtual Steering wheel -->
+  <link name="virtual_steer_link">
+    <visual>
+      <origin xyz="0.0 0.0 0.0" rpy="0.0 0.0 0.0" />
+      <geometry>
+        <box size="0.01 0.15 0.075" />
+      </geometry>
+      <material name="">
+        <color rgba="1.0 1.0 0.0 1" />
+      </material>
+    </visual>
+    <inertial>  <!-- Gazebo won't show this link without this inertial mass -->
+      <origin xyz="0.0 0.0 0.0" rpy="0.0 0.0 0.0" />
+      <mass value="0.001" />
+      <inertia ixx="0.0" ixy="0.0" ixz="0.0" iyy="0.0" iyz="0.0" izz="0.0" />
+    </inertial>
+  </link>
+  <joint name="virtual_steering_wheel_joint" type="revolute">
+    <origin xyz="-0.32 0.0 0.0" rpy="0.0 0.0 0.0" />
+    <parent link="base_link" />
+    <child link="virtual_steer_link" />
+    <axis xyz="-1 0 0" />
+    <limit lower="-3" upper="3" effort="200" velocity="20" />
+  </joint>
 </robot>

File: nav2_bringup/tarkbot_model/tarkbot_move.urdf.xacro (robot description, xacro)
@@ -24,8 +24,62 @@
   </ros2_control>
   <gazebo>
-    <plugin name="gazebo_ros2_control" filename="libgazebo_ros2_control.so">
-      <parameters>
-        $(find nav2_bringup)/params/ackermann_drive_controller.yaml
-      </parameters>
+    <plugin name="gazebo_ros_joint_state_publisher"
+      filename="libgazebo_ros_joint_state_publisher.so">
+      <update_rate>100</update_rate>
+      <joint_name>left_back_wheel_joint</joint_name>
+      <joint_name>right_back_wheel_joint</joint_name>
+      <joint_name>left_front_steering_joint</joint_name>
+      <joint_name>right_front_steering_joint</joint_name>
+      <joint_name>left_front_wheel_joint</joint_name>
+      <joint_name>right_front_wheel_joint</joint_name>
+      <joint_name>virtual_steering_wheel_joint</joint_name>
+    </plugin>
+  </gazebo>
+  <gazebo>
+    <plugin name="gazebo_ros_joint_pose_trajectory"
+      filename="libgazebo_ros_joint_pose_trajectory.so">
+      <update_rate>2</update_rate>
+    </plugin>
+  </gazebo>
+  <gazebo>
+    <plugin name='gazebo_ackermann_drive' filename='libgazebo_ros_ackermann_drive.so'>
+      <ros>
+        <!-- <namespace>ugv_gazebo_ackermann</namespace> -->
+        <remapping>cmd_vel:=cmd_vel</remapping>
+        <remapping>odom:=odom</remapping>
+        <remapping>distance:=distance</remapping>
+      </ros>
+      <update_rate>100.0</update_rate>
+      <!-- wheels -->
+      <front_left_joint>left_front_wheel_joint</front_left_joint>
+      <front_right_joint>right_front_wheel_joint</front_right_joint>
+      <rear_left_joint>left_back_wheel_joint</rear_left_joint>
+      <rear_right_joint>right_back_wheel_joint</rear_right_joint>
+      <left_steering_joint>left_front_steering_joint</left_steering_joint>
+      <right_steering_joint>right_front_steering_joint</right_steering_joint>
+      <steering_wheel_joint>virtual_steering_wheel_joint</steering_wheel_joint>
+      <!-- Max absolute steer angle for tyre in radians-->
+      <!-- Any cmd_vel angular z greater than this would be capped -->
+      <max_steer>0.383972</max_steer>
+      <!-- Max absolute steering angle of steering wheel -->
+      <max_steering_angle>1.570796</max_steering_angle>
+      <!-- Max absolute linear speed in m/s -->
+      <max_speed>5</max_speed>
+      <!-- PID tuning -->
+      <left_steering_pid_gain>1500 0 1</left_steering_pid_gain>
+      <left_steering_i_range>0 0</left_steering_i_range>
+      <right_steering_pid_gain>1500 0 1</right_steering_pid_gain>
+      <right_steering_i_range>0 0</right_steering_i_range>
+      <linear_velocity_pid_gain>1500 0 1</linear_velocity_pid_gain>
+      <linear_velocity_i_range>0 0</linear_velocity_i_range>
+      <!-- output -->
+      <publish_odom>true</publish_odom>
+      <publish_odom_tf>true</publish_odom_tf>     <!-- Don't pubslish this when using robot
+          localization -->
+      <publish_wheel_tf>false</publish_wheel_tf>  <!-- Don't publish this. It will override all
+          wheel frames to robot_base_frame parameter below.-->
+      <publish_distance>true</publish_distance>
+      <odometry_frame>odom</odometry_frame>
+      <robot_base_frame>base_footprint</robot_base_frame>
     </plugin>
   </gazebo>
